File: Electronics/string_lights_revA.brd (EAGLE design)
At the start: 185.9 x 119.9 mm, 25 parts, among them U1 ESP32-ADAPTER

Commit message: Electronics: finished RevA
Parts:
- removed C4: (no value), 1_domaci:ELYT-10MM
- added C5: 100nF, 1_domaci:C0805
- added R12, R13: 10k, 1_domaci:R0805
- added T1: BSS138, 1_domaci:SOT23
- C1, C2: value (none) -> 10uF
- C3: value (none) -> 470uF
- R1, R4: value 1k -> 15k
- R2, R5: value 1k -> 6k8
- R3, R6: value 1k -> 10k
- U2: value (none) -> AMS1117
- moved C1 52.8 mm to (16.3, 31.4)
- moved C2 52.8 mm to (16.3, 40.5)
- moved U2 52.8 mm to (13.8, 35.9)
- moved C3 50.4 mm to (16.0, 27.1), turned to 0 degrees
- moved R8 36.1 mm to (17.3, 20.4)
- moved JP4 36.0 mm to (18.5, 13.3)
- moved R7 36.0 mm to (19.8, 20.4)
- moved R9 34.8 mm to (12.2, 20.4)
- moved R10 34.6 mm to (9.65, 20.4)
- moved JP1 34.5 mm to (10.9, 13.3)
- moved JP8 32.7 mm to (12.4, 56.5)
- moved R5 29.6 mm to (47.8, 20.3)
- moved R6 27.9 mm to (42.7, 20.3)
- moved JP3 27.7 mm to (43.9, 13.3)
- moved JP7 24.7 mm to (37.5, 56.5)
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Connections:
- removed net N$3 (its old number): JP2.2, R2.2
- removed net N$6 (its old number): JP3.2, R5.2
- new net N$12: JP8.2, R12.1, T1.3
- new net N$4: JP2.1, R2.2
- new net N$7: JP3.4, R4.2
- net +3V3: now also R13.2, T1.1; no longer C4.P
- net +5V: now also C5.2, JP5.2, R12.2; no longer JP5.1
- net AP_SWITCH: now also U1.21
- net BUTTON1: now also U1.29
- net BUTTON2: now also U1.30
- net GND: now also C5.1, JP2.2, JP3.2, JP6.1; no longer C4.N, JP2.4, JP3.4, JP6.2
- net LED1_B: now also U1.10
- net LED1_G: now also U1.9
- net LED1_R: now also U1.11
- net LED2_B: now also U1.7
- net LED2_G: now also U1.6
- net LED2_R: now also U1.8
- net LED_DATA: now also R13.1, T1.2; no longer JP8.2
- net N$1: now also JP5.1, JP6.2; no longer JP5.2, JP6.1
- net N$2: now also JP2.4; no longer JP2.1
- net N$5: now also R5.2; no longer R4.2
Routing:
- net GND: track 0.00 -> 219.4 mm
- net +5V: track 0.00 -> 108.0 mm
- net +3V3: track 0.00 -> 85.9 mm, vias 0 -> 2
- net N$1: track 0.00 -> 35.6 mm
- net LED1_R: track 0.00 -> 32.9 mm
- net LED1_B: track 0.00 -> 29.3 mm
- net LED_DATA: track 0.00 -> 25.9 mm
- net LED1_G: track 0.00 -> 23.1 mm
- net LED2_R: track 0.00 -> 18.2 mm
- net N$12: track 0.00 -> 15.6 mm
- net LED2_B: track 0.00 -> 14.6 mm
- net BUTTON1: track 0.00 -> 13.7 mm
- net N$10: track 0.00 -> 12.1 mm
- net LED2_G: track 0.00 -> 9.96 mm
- net AP_SWITCH: track 0.00 -> 9.36 mm
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Other:
- board size 185.9 x 119.9 mm -> 100.7 x 120.9 mm
- board text added: "+3V3"
- board text added: "+5V"
- board text added: "AP_SW"
- board text added: "B"
- board text added: "B1"
- board text added: "B2"
- board text added: "DATA"
- board text added: "G"
- board text added: "Gr"
- board text added: "PWR_SW"
- board text added: "R"
